File: armm0/armm0.sch (KiCad schematic (older format))
At the start: 10 parts

Commit message: board: Everything is upside down
Signed-off-by: Ben <bdl@live.co.uk>
Parts:
- C1: renamed from 0.1uF; value C -> 100nF; footprint (none) -> Capacitor_THT:CP_Radial_D4.0mm_P2.00mm
- C2: renamed from 4.7uF; value C -> 4.7uF; footprint (none) -> Capacitor_SMD:C_1206_3216Metric
- C3: renamed from 1nF; value C -> 1uf; footprint (none) -> Capacitor_SMD:C_1206_3216Metric
- J1: renamed from J?; footprint (none) -> Connector_IDC:IDC-Header_2x10_P2.54mm_Vertical
- J2, J3: renamed from J?; footprint (none) -> Connector_PinHeader_2.54mm:PinHeader_2x24_P2.54mm_Vertical
- R1, R2: renamed from 4.7k; value R -> 4.7k; footprint (none) -> Resistor_SMD:R_1206_3216Metric
- gave numbers to parts that had none: 2
Connections:
- wire segments 21 -> 22
Other:
- note added: "ceramic"
Changed lines of the file:
@@
 $EndDescr
 $Comp
-L MCU_ST_STM32F0:STM32F070F6Px U?
+L MCU_ST_STM32F0:STM32F070F6Px U1
 U 1 1 5B61CC97
 P 3300 2700
-F 0 "U?" H 3200 2750 50  0000 C CNN
+F 0 "U1" H 3200 2750 50  0000 C CNN
 F 1 "STM32F070F6Px" H 3200 2650 50  0000 C CNN
 F 2 "Package_SO:TSSOP-20_4.4x6.5mm_P0.65mm" H 2700 2000 50  0001 R CNN
@@
 $EndComp
 $Comp
-L power:GND #PWR?
+L power:GND #PWR0101
 U 1 1 5B61CD19
-P 3100 3500
-F 0 "#PWR?" H 3100 3250 50  0001 C CNN
-F 1 "GND" H 3105 3327 50  0000 C CNN
-F 2 "" H 3100 3500 50  0001 C CNN
-F 3 "" H 3100 3500 50  0001 C CNN
-	1    3100 3500
-	1    0    0    -1
-$EndComp
-$Comp
-L Connector_Generic:Conn_02x10_Odd_Even J?
+P 3100 3550
+F 0 "#PWR0101" H 3100 3300 50  0001 C CNN
+F 1 "GND" H 3105 3377 50  0000 C CNN
+F 2 "" H 3100 3550 50  0001 C CNN
+F 3 "" H 3100 3550 50  0001 C CNN
+	1    3100 3550
+	1    0    0    -1
+$EndComp
+$Comp
+L Connector_Generic:Conn_02x10_Odd_Even J1
 U 1 1 5B61CEB8
 P 5750 2700
-F 0 "J?" H 5800 3317 50  0000 C CNN
+F 0 "J1" H 5800 3317 50  0000 C CNN
 F 1 "Conn_02x10_Odd_Even" H 5800 3226 50  0000 C CNN
-F 2 "" H 5750 2700 50  0001 C CNN
+F 2 "Connector_IDC:IDC-Header_2x10_P2.54mm_Vertical" H 5750 2700 50  0001 C CNN
 F 3 "~" H 5750 2700 50  0001 C CNN
 	1    5750 2700
@@
 $EndComp
 $Comp
-L power:GND #PWR?
+L power:GND #PWR0102
 U 1 1 5B61CF3E
 P 2350 2450
-F 0 "#PWR?" H 2350 2200 50  0001 C CNN
+F 0 "#PWR0102" H 2350 2200 50  0001 C CNN
 F 1 "GND" H 2355 2277 50  0000 C CNN
 F 2 "" H 2350 2450 50  0001 C CNN
@@
 NRST
 $Comp
-L power:+3V3 #PWR?
+L power:+3V3 #PWR0103
 U 1 1 5B61D1B3
 P 2850 1500
-F 0 "#PWR?" H 2850 1350 50  0001 C CNN
+F 0 "#PWR0103" H 2850 1350 50  0001 C CNN
 F 1 "+3V3" H 2865 1673 50  0000 C CNN
 F 2 "" H 2850 1500 50  0001 C CNN
@@
 $EndComp
 $Comp
-L power:+3V3 #PWR?
+L power:+3V3 #PWR0104
 U 1 1 5B61D1D9
 P 3400 1500
-F 0 "#PWR?" H 3400 1350 50  0001 C CNN
+F 0 "#PWR0104" H 3400 1350 50  0001 C CNN
 F 1 "+3V3" H 3415 1673 50  0000 C CNN
 F 2 "" H 3400 1500 50  0001 C CNN
@@
 $EndComp
 $Comp
-L Device:C 0.1uF
+L Device:C C1
 U 1 1 5B61D296
 P 2150 2000
-F 0 "0.1uF" H 2265 2046 50  0000 L CNN
-F 1 "C" H 2265 1955 50  0000 L CNN
-F 2 "" H 2188 1850 50  0001 C CNN
+F 0 "C1" H 2265 2046 50  0000 L CNN
+F 1 "100nF" H 2265 1955 50  0000 L CNN
+F 2 "Capacitor_THT:CP_Radial_D4.0mm_P2.00mm" H 2188 1850 50  0001 C CNN
 F 3 "~" H 2150 2000 50  0001 C CNN
 	1    2150 2000
@@
 	2600 2200 2400 2200
 $Comp
-L power:GND #PWR?
+L power:GND #PWR0105
 U 1 1 5B61D421
 P 2150 2150
-F 0 "#PWR?" H 2150 1900 50  0001 C CNN
+F 0 "#PWR0105" H 2150 1900 50  0001 C CNN
 F 1 "GND" H 2155 1977 50  0000 C CNN
 F 2 "" H 2150 2150 50  0001 C CNN
@@
 Connection ~ 2150 1850
 $Comp
-L Device:C 4.7uF
+L Device:C C2
 U 1 1 5B61DAE3
 P 2850 1650
-F 0 "4.7uF" H 2965 1696 50  0000 L CNN
-F 1 "C" H 2965 1605 50  0000 L CNN
-F 2 "" H 2888 1500 50  0001 C CNN
+F 0 "C2" H 2965 1696 50  0000 L CNN
+F 1 "4.7uF" H 2965 1605 50  0000 L CNN
+F 2 "Capacitor_SMD:C_1206_3216Metric" H 2888 1500 50  0001 C CNN
 F 3 "~" H 2850 1650 50  0001 C CNN
 	1    2850 1650
@@
 $EndComp
 $Comp
-L power:GND #PWR?
+L power:GND #PWR0106
 U 1 1 5B61DB19
 P 2850 1800
-F 0 "#PWR?" H 2850 1550 50  0001 C CNN
+F 0 "#PWR0106" H 2850 1550 50  0001 C CNN
 F 1 "GND" H 2855 1627 50  0000 C CNN
 F 2 "" H 2850 1800 50  0001 C CNN
@@
 	3100 1500 3100 2000
 $Comp
-L Device:C 1nF
+L Device:C C3
 U 1 1 5B61DBAF
 P 3400 1650
-F 0 "1nF" H 3515 1696 50  0000 L CNN
-F 1 "C" H 3515 1605 50  0000 L CNN
-F 2 "" H 3438 1500 50  0001 C CNN
+F 0 "C3" H 3515 1696 50  0000 L CNN
+F 1 "1uf" H 3515 1605 50  0000 L CNN
+F 2 "Capacitor_SMD:C_1206_3216Metric" H 3438 1500 50  0001 C CNN
 F 3 "~" H 3400 1650 50  0001 C CNN
 	1    3400 1650
@@
 Connection ~ 3400 1500
 $Comp
-L power:GND #PWR?
+L power:GND #PWR0107
 U 1 1 5B61DCB4
 P 3400 1800
-F 0 "#PWR?" H 3400 1550 50  0001 C CNN
+F 0 "#PWR0107" H 3400 1550 50  0001 C CNN
 F 1 "GND" H 3405 1627 50  0000 C CNN
 F 2 "" H 3400 1800 50  0001 C CNN
@@
 	2850 1500 3100 1500
 $Comp
-L Regulator_Linear:LD1117S33TR_SOT223 U?
+L Regulator_Linear:LD1117S33TR_SOT223 U2
 U 1 1 5B61E64C
 P 4900 1000
-F 0 "U?" H 4900 1242 50  0000 C CNN
+F 0 "U2" H 4900 1242 50  0000 C CNN
 F 1 "LD1117S33TR_SOT223" H 4900 1151 50  0000 C CNN
 F 2 "Package_TO_SOT_SMD:SOT-223-3_TabPin2" H 4900 1200 50  0001 C CNN
@@
 $EndComp
 $Comp
-L power:+5V #PWR?
+L power:+5V #PWR0108
 U 1 1 5B61EA0F
 P 5500 1000
-F 0 "#PWR?" H 5500 850 50  0001 C CNN
+F 0 "#PWR0108" H 5500 850 50  0001 C CNN
 F 1 "+5V" H 5515 1173 50  0000 C CNN
 F 2 "" H 5500 1000 50  0001 C CNN
@@
 	5200 1000 5500 1000
 $Comp
-L power:+3V3 #PWR?
+L power:+3V3 #PWR0109
 U 1 1 5B61EC5D
 P 4300 1000
-F 0 "#PWR?" H 4300 850 50  0001 C CNN
+F 0 "#PWR0109" H 4300 850 50  0001 C CNN
 F 1 "+3V3" H 4315 1173 50  0000 C CNN
 F 2 "" H 4300 1000 50  0001 C CNN
@@
 	4300 1000 4600 1000
 $Comp
-L power:GND #PWR?
+L power:GND #PWR0110
 U 1 1 5B61ED16
 P 4900 1300
-F 0 "#PWR?" H 4900 1050 50  0001 C CNN
+F 0 "#PWR0110" H 4900 1050 50  0001 C CNN
 F 1 "GND" H 4905 1127 50  0000 C CNN
 F 2 "" H 4900 1300 50  0001 C CNN
@@
 $EndComp
 $Comp
-L Connector_Generic:Conn_02x24_Odd_Even J?
+L Connector_Generic:Conn_02x24_Odd_Even J3
 U 1 1 5B61EE49
 P 10000 2100
-F 0 "J?" H 10050 3417 50  0000 C CNN
+F 0 "J3" H 10050 3417 50  0000 C CNN
 F 1 "Conn_02x24_Odd_Even" H 10050 3326 50  0000 C CNN
-F 2 "" H 10000 2100 50  0001 C CNN
+F 2 "Connector_PinHeader_2.54mm:PinHeader_2x24_P2.54mm_Vertical" H 10000 2100 50  0001 C CNN
 F 3 "~" H 10000 2100 50  0001 C CNN
 	1    10000 2100
@@
 $EndComp
 $Comp
-L Connector_Generic:Conn_02x24_Odd_Even J?
+L Connector_Generic:Conn_02x24_Odd_Even J2
 U 1 1 5B61EEC0
 P 8450 2100
-F 0 "J?" H 8500 3417 50  0000 C CNN
+F 0 "J2" H 8500 3417 50  0000 C CNN
 F 1 "Conn_02x24_Odd_Even" H 8500 3326 50  0000 C CNN
-F 2 "" H 8450 2100 50  0001 C CNN
+F 2 "Connector_PinHeader_2.54mm:PinHeader_2x24_P2.54mm_Vertical" H 8450 2100 50  0001 C CNN
 F 3 "~" H 8450 2100 50  0001 C CNN
 	1    8450 2100
@@
 AN\n
 $Comp
-L power:+5V #PWR?
+L power:+5V #PWR0111
 U 1 1 5B61F4F5
 P 9600 3300
-F 0 "#PWR?" H 9600 3150 50  0001 C CNN
+F 0 "#PWR0111" H 9600 3150 50  0001 C CNN
 F 1 "+5V" H 9615 3473 50  0000 C CNN
 F 2 "" H 9600 3300 50  0001 C CNN
@@
 I2C1_SCL
 $Comp
-L Device:R 4.7k
+L Device:R R1
 U 1 1 5B61FDAE
 P 1900 2800
-F 0 "4.7k" H 1970 2846 50  0000 L CNN
-F 1 "R" H 1970 2755 50  0000 L CNN
-F 2 "" V 1830 2800 50  0001 C CNN
+F 0 "R1" H 1970 2846 50  0000 L CNN
+F 1 "4.7k" H 1970 2755 50  0000 L CNN
+F 2 "Resistor_SMD:R_1206_3216Metric" V 1830 2800 50  0001 C CNN
 F 3 "~" H 1900 2800 50  0001 C CNN
 	1    1900 2800
@@
 $EndComp
 $Comp
-L Device:R 4.7k
+L Device:R R2
 U 1 1 5B61FEE2
 P 2150 2800
-F 0 "4.7k" H 2220 2846 50  0000 L CNN
-F 1 "R" H 2220 2755 50  0000 L CNN
-F 2 "" V 2080 2800 50  0001 C CNN
+F 0 "R2" H 2220 2846 50  0000 L CNN
+F 1 "4.7k" H 2220 2755 50  0000 L CNN
+F 2 "Resistor_SMD:R_1206_3216Metric" V 2080 2800 50  0001 C CNN
 F 3 "~" H 2150 2800 50  0001 C CNN
 	1    2150 2800
@@
 $EndComp
 $Comp
-L power:+3V3 #PWR?
+L power:+3V3 #PWR0112
 U 1 1 5B61FFC9
 P 1900 2600
-F 0 "#PWR?" H 1900 2450 50  0001 C CNN
+F 0 "#PWR0112" H 1900 2450 50  0001 C CNN
 F 1 "+3V3" H 1915 2773 50  0000 C CNN
 F 2 "" H 1900 2600 50  0001 C CNN
@@
 Text GLabel 6050 2400 2    50   Input ~ 0
 SWCLK
+Text Notes 3000 1450 0    50   Italic 0
+ceramic
+Wire Wire Line
+	3100 3500 3100 3550
 $EndSCHEMATC

Commit message: armm0: Add eagle project
Signed-off-by: Ben <bdl@live.co.uk>
Other:
- moved on the sheet: U2
Changed lines of the file:
@@
 EESchema Schematic File Version 4
+LIBS:armm0-cache
 EELAYER 26 0
 EELAYER END
@@
 L Regulator_Linear:LD1117S33TR_SOT223 U2
 U 1 1 5B61E64C
-P 4900 1000
-F 0 "U2" H 4900 1242 50  0000 C CNN
-F 1 "LD1117S33TR_SOT223" H 4900 1151 50  0000 C CNN
-F 2 "Package_TO_SOT_SMD:SOT-223-3_TabPin2" H 4900 1200 50  0001 C CNN
-F 3 "http://www.st.com/st-web-ui/static/active/en/resource/technical/document/datasheet/CD00000544.pdf" H 5000 750 50  0001 C CNN
-	1    4900 1000
+P 5350 950
+F 0 "U2" H 5350 1192 50  0000 C CNN
+F 1 "LD1117S33TR_SOT223" H 5350 1101 50  0000 C CNN
+F 2 "Package_TO_SOT_SMD:SOT-223-3_TabPin2" H 5350 1150 50  0001 C CNN
+F 3 "http://www.st.com/st-web-ui/static/active/en/resource/technical/document/datasheet/CD00000544.pdf" H 5450 700 50  0001 C CNN
+	1    5350 950
 	-1   0    0    -1
 $EndComp
@@
 L power:+5V #PWR0108
 U 1 1 5B61EA0F
-P 5500 1000
-F 0 "#PWR0108" H 5500 850 50  0001 C CNN
-F 1 "+5V" H 5515 1173 50  0000 C CNN
-F 2 "" H 5500 1000 50  0001 C CNN
-F 3 "" H 5500 1000 50  0001 C CNN
-	1    5500 1000
-	1    0    0    -1
-$EndComp
-Wire Wire Line
-	5200 1000 5500 1000
+P 5950 950
+F 0 "#PWR0108" H 5950 800 50  0001 C CNN
+F 1 "+5V" H 5965 1123 50  0000 C CNN
+F 2 "" H 5950 950 50  0001 C CNN
+F 3 "" H 5950 950 50  0001 C CNN
+	1    5950 950
+	1    0    0    -1
+$EndComp
+Wire Wire Line
+	5650 950  5950 950
 $Comp
 L power:+3V3 #PWR0109
 U 1 1 5B61EC5D
-P 4300 1000
-F 0 "#PWR0109" H 4300 850 50  0001 C CNN
-F 1 "+3V3" H 4315 1173 50  0000 C CNN
-F 2 "" H 4300 1000 50  0001 C CNN
-F 3 "" H 4300 1000 50  0001 C CNN
-	1    4300 1000
-	1    0    0    -1
-$EndComp
-Wire Wire Line
-	4300 1000 4600 1000
+P 4750 950
+F 0 "#PWR0109" H 4750 800 50  0001 C CNN
+F 1 "+3V3" H 4765 1123 50  0000 C CNN
+F 2 "" H 4750 950 50  0001 C CNN
+F 3 "" H 4750 950 50  0001 C CNN
+	1    4750 950
+	1    0    0    -1
+$EndComp
+Wire Wire Line
+	4750 950  5050 950
 $Comp
 L power:GND #PWR0110
 U 1 1 5B61ED16
-P 4900 1300
-F 0 "#PWR0110" H 4900 1050 50  0001 C CNN
-F 1 "GND" H 4905 1127 50  0000 C CNN
-F 2 "" H 4900 1300 50  0001 C CNN
-F 3 "" H 4900 1300 50  0001 C CNN
-	1    4900 1300
+P 5350 1250
+F 0 "#PWR0110" H 5350 1000 50  0001 C CNN
+F 1 "GND" H 5355 1077 50  0000 C CNN
+F 2 "" H 5350 1250 50  0001 C CNN
+F 3 "" H 5350 1250 50  0001 C CNN
+	1    5350 1250
 	1    0    0    -1
 $EndComp
@@
 Wire Wire Line
 	3100 3500 3100 3550
+Wire Notes Line width 12
+	4450 3850 950  3850
+Wire Notes Line width 12
+	950  3850 950  900
+Wire Notes Line width 12
+	950  900  4450 900
+Wire Notes Line width 12
+	4450 900  4450 3850
+Wire Notes Line width 12
+	5100 1850 6600 1850
+Wire Notes Line width 12
+	6600 1850 6600 3350
+Wire Notes Line width 12
+	6600 3350 5100 3350
+Wire Notes Line width 12
+	5100 3350 5100 1850
+Wire Notes Line width 12
+	7900 600  10750 600
+Wire Notes Line width 12
+	10750 600  10750 3650
+Wire Notes Line width 12
+	10750 3650 7900 3650
+Wire Notes Line width 12
+	7900 3650 7900 600
 $EndSCHEMATC

Commit message: sch: Add Conn_02x08 for shorter board
Signed-off-by: Ben Lancaster <bdl@live.co.uk>
Parts:
- added J4, J5: Conn_02x08_Odd_Even, symbol Connector_Generic:Conn_02x08_Odd_Even
- C1: footprint Capacitor_THT:CP_Radial_D4.0mm_P2.00mm -> Capacitor_SMD:C_1206_3216Metric_Pad1.42x1.75mm_HandSolder
- C2, C3: footprint Capacitor_SMD:C_1206_3216Metric -> Capacitor_SMD:C_1206_3216Metric_Pad1.42x1.75mm_HandSolder
Connections:
- net labels added: +3.3V, ADC_IN0, ADC_IN1, C0, C1, C10, C11, C2, C3, C4, C5, C6, C7, C8, C9
- wire segments 22 -> 26
Changed lines of the file:
@@
 F 0 "C1" H 2265 2046 50  0000 L CNN
 F 1 "100nF" H 2265 1955 50  0000 L CNN
-F 2 "Capacitor_THT:CP_Radial_D4.0mm_P2.00mm" H 2188 1850 50  0001 C CNN
+F 2 "Capacitor_SMD:C_1206_3216Metric_Pad1.42x1.75mm_HandSolder" H 2188 1850 50  0001 C CNN
 F 3 "~" H 2150 2000 50  0001 C CNN
 	1    2150 2000
@@
 F 0 "C2" H 2965 1696 50  0000 L CNN
 F 1 "4.7uF" H 2965 1605 50  0000 L CNN
-F 2 "Capacitor_SMD:C_1206_3216Metric" H 2888 1500 50  0001 C CNN
+F 2 "Capacitor_SMD:C_1206_3216Metric_Pad1.42x1.75mm_HandSolder" H 2888 1500 50  0001 C CNN
 F 3 "~" H 2850 1650 50  0001 C CNN
 	1    2850 1650
@@
 F 0 "C3" H 3515 1696 50  0000 L CNN
 F 1 "1uf" H 3515 1605 50  0000 L CNN
-F 2 "Capacitor_SMD:C_1206_3216Metric" H 3438 1500 50  0001 C CNN
+F 2 "Capacitor_SMD:C_1206_3216Metric_Pad1.42x1.75mm_HandSolder" H 3438 1500 50  0001 C CNN
 F 3 "~" H 3400 1650 50  0001 C CNN
 	1    3400 1650
@@
 Wire Notes Line width 12
 	7900 3650 7900 600
+Text GLabel 3900 2200 2    50   Input ~ 0
+ADC_IN0
+Text GLabel 3900 2300 2    50   Input ~ 0
+ADC_IN1
+$Comp
+L Connector_Generic:Conn_02x08_Odd_Even J4
+U 1 1 5B65C2FA
+P 8450 4350
+F 0 "J4" H 8500 4867 50  0000 C CNN
+F 1 "Conn_02x08_Odd_Even" H 8500 4776 50  0000 C CNN
+F 2 "" H 8450 4350 50  0001 C CNN
+F 3 "~" H 8450 4350 50  0001 C CNN
+	1    8450 4350
+	1    0    0    -1
+$EndComp
+$Comp
+L Connector_Generic:Conn_02x08_Odd_Even J5
+U 1 1 5B65C3B3
+P 10000 4300
+F 0 "J5" H 10050 4817 50  0000 C CNN
+F 1 "Conn_02x08_Odd_Even" H 10050 4726 50  0000 C CNN
+F 2 "" H 10000 4300 50  0001 C CNN
+F 3 "~" H 10000 4300 50  0001 C CNN
+	1    10000 4300
+	1    0    0    -1
+$EndComp
+$Comp
+L power:+5V #PWR02
+U 1 1 5B65C5B4
+P 9500 4700
+F 0 "#PWR02" H 9500 4550 50  0001 C CNN
+F 1 "+5V" H 9515 4873 50  0000 C CNN
+F 2 "" H 9500 4700 50  0001 C CNN
+F 3 "" H 9500 4700 50  0001 C CNN
+	1    9500 4700
+	1    0    0    -1
+$EndComp
+$Comp
+L power:GND #PWR04
+U 1 1 5B65D123
+P 10500 4700
+F 0 "#PWR04" H 10500 4450 50  0001 C CNN
+F 1 "GND" H 10505 4527 50  0000 C CNN
+F 2 "" H 10500 4700 50  0001 C CNN
+F 3 "" H 10500 4700 50  0001 C CNN
+	1    10500 4700
+	1    0    0    -1
+$EndComp
+Wire Wire Line
+	10500 4700 10300 4700
+$Comp
+L power:GND #PWR01
+U 1 1 5B65D460
+P 9350 4300
+F 0 "#PWR01" H 9350 4050 50  0001 C CNN
+F 1 "GND" H 9355 4127 50  0000 C CNN
+F 2 "" H 9350 4300 50  0001 C CNN
+F 3 "" H 9350 4300 50  0001 C CNN
+	1    9350 4300
+	1    0    0    -1
+$EndComp
+$Comp
+L power:+3.3V #PWR03
+U 1 1 5B65D7DC
+P 10600 4300
+F 0 "#PWR03" H 10600 4150 50  0001 C CNN
+F 1 "+3.3V" H 10615 4473 50  0000 C CNN
+F 2 "" H 10600 4300 50  0001 C CNN
+F 3 "" H 10600 4300 50  0001 C CNN
+	1    10600 4300
+	1    0    0    -1
+$EndComp
+Text GLabel 9800 4000 0    50   Input ~ 0
+C0
+Text GLabel 10300 4000 2    50   Input ~ 0
+C1
+Text GLabel 9800 4100 0    50   Input ~ 0
+C2
+Text GLabel 9800 4200 0    50   Input ~ 0
+C4
+Text GLabel 10300 4100 2    50   Input ~ 0
+C3
+Text GLabel 10300 4200 2    50   Input ~ 0
+C5
+Text GLabel 10300 4400 2    50   Input ~ 0
+C7
+Text GLabel 10300 4500 2    50   Input ~ 0
+C9
+Text GLabel 10300 4600 2    50   Input ~ 0
+C11
+Text GLabel 9800 4400 0    50   Input ~ 0
+C6
+Text GLabel 9800 4500 0    50   Input ~ 0
+C8
+Text GLabel 9800 4600 0    50   Input ~ 0
+C10
+Wire Wire Line
+	9500 4700 9800 4700
+Wire Wire Line
+	9350 4300 9800 4300
+Wire Wire Line
+	10300 4300 10600 4300
 $EndSCHEMATC

Commit message: sch: Add footprints for Conn_02x08
Signed-off-by: Ben Lancaster <bdl@live.co.uk>
Parts:
- J4, J5: footprint (none) -> Connector_PinHeader_2.54mm:PinHeader_2x08_P2.54mm_Vertical
Changed lines of the file:
@@
 F 0 "J4" H 8500 4867 50  0000 C CNN
 F 1 "Conn_02x08_Odd_Even" H 8500 4776 50  0000 C CNN
-F 2 "" H 8450 4350 50  0001 C CNN
+F 2 "Connector_PinHeader_2.54mm:PinHeader_2x08_P2.54mm_Vertical" H 8450 4350 50  0001 C CNN
 F 3 "~" H 8450 4350 50  0001 C CNN
 	1    8450 4350
@@
 F 0 "J5" H 10050 4817 50  0000 C CNN
 F 1 "Conn_02x08_Odd_Even" H 10050 4726 50  0000 C CNN
-F 2 "" H 10000 4300 50  0001 C CNN
+F 2 "Connector_PinHeader_2.54mm:PinHeader_2x08_P2.54mm_Vertical" H 10000 4300 50  0001 C CNN
 F 3 "~" H 10000 4300 50  0001 C CNN
 	1    10000 4300

Commit message: sch: stlink: Update stlink pinout
Signed-off-by: Ben Lancaster <bdl@live.co.uk>
Connections:
- net labels added: JTAG_TDI, JTAG_TDO, JTAG_TRST
- wire segments 26 -> 52
- no-connect marks 0 -> 2
Changed lines of the file:
@@
 P 5750 2700
 F 0 "J1" H 5800 3317 50  0000 C CNN
-F 1 "Conn_02x10_Odd_Even" H 5800 3226 50  0000 C CNN
+F 1 "Conn_02x10_Odd_Even" H 5850 3250 50  0000 C CNN
 F 2 "Connector_IDC:IDC-Header_2x10_P2.54mm_Vertical" H 5750 2700 50  0001 C CNN
 F 3 "~" H 5750 2700 50  0001 C CNN
@@
 Wire Wire Line
 	2150 3100 1700 3100
-Text GLabel 6050 2500 2    50   Input ~ 0
-I2C1_SDA
-Text GLabel 6050 2600 2    50   Input ~ 0
-I2C1_SCL
 Text Notes 2850 1150 0    50   ~ 10
 STM32F070F6
@@
 Text GLabel 3900 3200 2    50   Input ~ 0
 SWDIO
-Text GLabel 6050 2300 2    50   Input ~ 0
+Text GLabel 5550 2600 0    50   Input ~ 0
 SWDIO
-Text GLabel 6050 2400 2    50   Input ~ 0
+Text GLabel 5550 2700 0    50   Input ~ 0
 SWCLK
 Text Notes 3000 1450 0    50   Italic 0
@@
 Wire Notes Line width 12
 	4450 900  4450 3850
-Wire Notes Line width 12
-	5100 1850 6600 1850
-Wire Notes Line width 12
-	6600 1850 6600 3350
-Wire Notes Line width 12
-	6600 3350 5100 3350
-Wire Notes Line width 12
-	5100 3350 5100 1850
 Wire Notes Line width 12
 	7900 600  10750 600
@@
 Wire Wire Line
 	10300 4300 10600 4300
+Text GLabel 9350 5350 0    50   Input ~ 0
+C9
+Text GLabel 9600 5250 2    50   Input ~ 0
+I2C1_SDA
+Wire Wire Line
+	9350 5350 9600 5350
+Text GLabel 9350 5250 0    50   Input ~ 0
+C7
+Text GLabel 9600 5350 2    50   Input ~ 0
+I2C1_SCL
+Wire Wire Line
+	9350 5250 9600 5250
+$Comp
+L power:+3.3V #PWR?
+U 1 1 5B664D18
+P 5100 2300
+F 0 "#PWR?" H 5100 2150 50  0001 C CNN
+F 1 "+3.3V" H 5115 2473 50  0000 C CNN
+F 2 "" H 5100 2300 50  0001 C CNN
+F 3 "" H 5100 2300 50  0001 C CNN
+	1    5100 2300
+	1    0    0    -1
+$EndComp
+$Comp
+L power:GND #PWR?
+U 1 1 5B6659EA
+P 6200 2400
+F 0 "#PWR?" H 6200 2150 50  0001 C CNN
+F 1 "GND" V 6205 2272 50  0000 R CNN
+F 2 "" H 6200 2400 50  0001 C CNN
+F 3 "" H 6200 2400 50  0001 C CNN
+	1    6200 2400
+	0    -1   -1   0
+$EndComp
+Wire Wire Line
+	6050 2400 6100 2400
+Wire Wire Line
+	6050 2500 6100 2500
+Wire Wire Line
+	6100 2500 6100 2400
+Connection ~ 6100 2400
+Wire Wire Line
+	6100 2400 6200 2400
+Wire Wire Line
+	6050 2600 6100 2600
+Wire Wire Line
+	6100 2600 6100 2500
+Connection ~ 6100 2500
+Wire Wire Line
+	6050 2700 6100 2700
+Wire Wire Line
+	6100 2700 6100 2600
+Connection ~ 6100 2600
+Wire Wire Line
+	6050 2800 6100 2800
+Wire Wire Line
+	6100 2800 6100 2700
+Connection ~ 6100 2700
+Wire Wire Line
+	6050 2900 6100 2900
+Wire Wire Line
+	6100 2900 6100 2800
+Connection ~ 6100 2800
+Wire Wire Line
+	6050 3000 6100 3000
+Wire Wire Line
+	6100 3000 6100 2900
+Connection ~ 6100 2900
+Wire Wire Line
+	6050 3100 6100 3100
+Wire Wire Line
+	6100 3100 6100 3000
+Connection ~ 6100 3000
+Wire Wire Line
+	6050 3200 6100 3200
+Wire Wire Line
+	6100 3200 6100 3100
+Connection ~ 6100 3100
+Text GLabel 5550 3000 0    50   Input ~ 0
+NRST
+NoConn ~ 5550 2800
+NoConn ~ 5550 3100
+Wire Wire Line
+	5100 2300 5100 3200
+Text GLabel 5550 2400 0    50   Input ~ 0
+JTAG_TRST
+Text GLabel 5550 2500 0    50   Input ~ 0
+JTAG_TDO
+Wire Wire Line
+	5100 3200 5550 3200
+Wire Wire Line
+	5100 2300 5550 2300
+Connection ~ 5100 2300
+Text GLabel 5550 2900 0    50   Input ~ 0
+JTAG_TDI
+Wire Wire Line
+	6050 2300 6050 2200
+Wire Wire Line
+	6050 2200 5550 2200
+Wire Wire Line
+	5550 2200 5550 2300
+Connection ~ 5550 2300
 $EndSCHEMATC

Commit message: sch: Flip Conn_02x08 pin headers for upside down insertion to master board
Signed-off-by: Ben Lancaster <bdl@live.co.uk>
Connections:
- net labels added: F0, F1, F10, F11, F2, F3, F4, F5, F6, F7, F8, F9
- wire segments 52 -> 56

Commit message: sch: Switch between board or stlink power source with 3pin selector
Signed-off-by: Ben Lancaster <bdl@live.co.uk>
Parts:
- added D1, D2, D3, D4, D5: LED, LED_SMD:LED_1206_3216Metric_Pad1.42x1.75mm_HandSolder, symbol Device:LED
- added J6, J7: Conn_01x05_Male, Connector_PinHeader_2.54mm:PinHeader_1x05_P2.54mm_Vertical, symbol Connector:Conn_01x05_Male
- added J8: Conn_01x03_Male, Connector_PinHeader_2.54mm:PinHeader_1x03_P2.54mm_Vertical, symbol Connector:Conn_01x03_Male
- added R3, R4, R5, R6, R7: R, Resistor_SMD:R_1206_3216Metric_Pad1.42x1.75mm_HandSolder, symbol Device:R
Connections:
- net labels added: BOARD_3V3, STLINK_3V3
- wire segments 56 -> 67
- no-connect marks 2 -> 9
Other:
- note added: "Active LOW"
- note added: "MCU_DEBUG_LEDS"
- note added: "PWR_GOOD"
- note added: "Power source selector"

Commit message: pcb: Some wiring done
Signed-off-by: Ben Lancaster <bdl@live.co.uk>
Connections:
- net labels added: FPGA_3V3
- wire segments 67 -> 65
- no-connect marks 9 -> 16
Changed lines of the file:
@@
-	1    0    0    -1
-$EndComp
-$Comp
-L power:+3.3V #PWR03
-U 1 1 5B65D7DC
-P 10550 4450
-F 0 "#PWR03" H 10550 4300 50  0001 C CNN
-F 1 "+3.3V" H 10565 4623 50  0000 C CNN
-F 2 "" H 10550 4450 50  0001 C CNN
-F 3 "" H 10550 4450 50  0001 C CNN
-	1    10550 4450
 	1    0    0    -1
 $EndComp
@@
 Wire Wire Line
 	9300 4450 9750 4450
-Wire Wire Line
-	10250 4450 10550 4450
 Text GLabel 9750 5350 0    50   Input ~ 0
 C9
@@
 	8700 4600 8950 4600
 $Comp
-L power:+3.3V #PWR0116
-U 1 1 5B67F6F6
-P 7850 4600
-F 0 "#PWR0116" H 7850 4450 50  0001 C CNN
-F 1 "+3.3V" H 7865 4773 50  0000 C CNN
-F 2 "" H 7850 4600 50  0001 C CNN
-F 3 "" H 7850 4600 50  0001 C CNN
-	1    7850 4600
-	1    0    0    -1
-$EndComp
-Wire Wire Line
-	7850 4600 8200 4600
-$Comp
 L power:+3.3V #PWR0117
 U 1 1 5B6804D1
@@
 Text GLabel 8100 5300 0    50   Input ~ 0
 F2
-Text GLabel 8400 5200 2    50   Input ~ 0
+Text GLabel 8550 5200 2    50   Input ~ 0
 ADC_IN0
-Text GLabel 8400 5300 2    50   Input ~ 0
+Text GLabel 8550 5300 2    50   Input ~ 0
 ADC_IN1
 Wire Wire Line
@@
 Text GLabel 6800 4250 0    50   Input ~ 0
 USART1_RX
+Text GLabel 6800 4450 0    50   Input ~ 0
+I2C1_SDA
 Text GLabel 6800 4350 0    50   Input ~ 0
-I2C1_SDA
-Text GLabel 6800 4450 0    50   Input ~ 0
 I2C1_SCL
 $Comp
@@
 Text Notes 6450 950  0    50   ~ 0
 Power source selector
+Text GLabel 8100 4600 0    50   Input ~ 0
+FPGA_3V3
+Text GLabel 10350 4450 2    50   Input ~ 0
+FPGA_3V3
+$Comp
+L power:+3V3 #PWR0116
+U 1 1 5B6BD2D4
+P 2450 4450
+F 0 "#PWR0116" H 2450 4300 50  0001 C CNN
+F 1 "+3V3" H 2465 4623 50  0000 C CNN
+F 2 "" H 2450 4450 50  0001 C CNN
+F 3 "" H 2450 4450 50  0001 C CNN
+	1    2450 4450
+	1    0    0    -1
+$EndComp
+$Comp
+L power:+3V3 #PWR0122
+U 1 1 5B6BD35C
+P 2750 4450
+F 0 "#PWR0122" H 2750 4300 50  0001 C CNN
+F 1 "+3V3" H 2765 4623 50  0000 C CNN
+F 2 "" H 2750 4450 50  0001 C CNN
+F 3 "" H 2750 4450 50  0001 C CNN
+	1    2750 4450
+	1    0    0    -1
+$EndComp
+$Comp
+L power:+3V3 #PWR0123
+U 1 1 5B6BD3EF
+P 3050 4450
+F 0 "#PWR0123" H 3050 4300 50  0001 C CNN
+F 1 "+3V3" H 3065 4623 50  0000 C CNN
+F 2 "" H 3050 4450 50  0001 C CNN
+F 3 "" H 3050 4450 50  0001 C CNN
+	1    3050 4450
+	1    0    0    -1
+$EndComp
+$Comp
+L power:+3V3 #PWR0124
+U 1 1 5B6BD42C
+P 3350 4450
+F 0 "#PWR0124" H 3350 4300 50  0001 C CNN
+F 1 "+3V3" H 3365 4623 50  0000 C CNN
+F 2 "" H 3350 4450 50  0001 C CNN
+F 3 "" H 3350 4450 50  0001 C CNN
+	1    3350 4450
+	1    0    0    -1
+$EndComp
+NoConn ~ 3900 2200
+NoConn ~ 3900 2300
+NoConn ~ 8400 5200
+NoConn ~ 8400 5300
+NoConn ~ 8300 4150
+NoConn ~ 8200 4600
+NoConn ~ 10250 4450
 $EndSCHEMATC
