File: armm0/armm0.sch (KiCad schematic (older format))
At the start: 25 parts, among them J1 Conn_02x10_Odd_Even, J2 Conn_02x24_Odd_Even, J3 Conn_02x24_Odd_Even, J4 Conn_02x08_Odd_Even, J5 Conn_02x08_Odd_Even, J6 Conn_01x05_Male, J7 Conn_01x05_Male, J8 Conn_01x03_Male, U1 STM32F070F6Px, U2 LD1117S33TR_SOT223

Commit message: pcb: Update
Signed-off-by: Ben Lancaster <bdl@live.co.uk>
Connections:
- net labels removed: C7, C9
- wire segments 65 -> 63
Changed lines of the file:
@@
 Text GLabel 10250 4350 2    50   Input ~ 0
 C5
-Text GLabel 10250 4550 2    50   Input ~ 0
-C7
-Text GLabel 10250 4650 2    50   Input ~ 0
-C9
 Text GLabel 10250 4750 2    50   Input ~ 0
 C11
@@
 Wire Wire Line
 	9300 4450 9750 4450
-Text GLabel 9750 5350 0    50   Input ~ 0
-C9
-Text GLabel 10000 5250 2    50   Input ~ 0
+Text GLabel 10250 4550 2    50   Input ~ 0
 I2C1_SDA
-Wire Wire Line
-	9750 5350 10000 5350
-Text GLabel 9750 5250 0    50   Input ~ 0
-C7
-Text GLabel 10000 5350 2    50   Input ~ 0
+Text GLabel 10250 4650 2    50   Input ~ 0
 I2C1_SCL
-Wire Wire Line
-	9750 5250 10000 5250
 $Comp
 L power:GND #PWR0114

Commit message: sch: Use resistor array for debug leds
Signed-off-by: Ben Lancaster <bdl@live.co.uk>
Parts:
- removed R4, R5, R6, R7: R, Resistor_SMD:R_1206_3216Metric_Pad1.42x1.75mm_HandSolder, symbol Device:R
- added RN1: R_Network04, Resistor_SMD:R_Array_Convex_4x1206, symbol Device:R_Network04
- R1, R2: footprint Resistor_SMD:R_1206_3216Metric -> Resistor_SMD:R_1206_3216Metric_Pad1.42x1.75mm_HandSolder
Connections:
- wire segments 63 -> 73
Changed lines of the file:
@@
 F 0 "R1" H 1970 2846 50  0000 L CNN
 F 1 "4.7k" H 1970 2755 50  0000 L CNN
-F 2 "Resistor_SMD:R_1206_3216Metric" V 1830 2800 50  0001 C CNN
+F 2 "Resistor_SMD:R_1206_3216Metric_Pad1.42x1.75mm_HandSolder" V 1830 2800 50  0001 C CNN
 F 3 "~" H 1900 2800 50  0001 C CNN
 	1    1900 2800
@@
 F 0 "R2" H 2220 2846 50  0000 L CNN
 F 1 "4.7k" H 2220 2755 50  0000 L CNN
-F 2 "Resistor_SMD:R_1206_3216Metric" V 2080 2800 50  0001 C CNN
+F 2 "Resistor_SMD:R_1206_3216Metric_Pad1.42x1.75mm_HandSolder" V 2080 2800 50  0001 C CNN
 F 3 "~" H 2150 2800 50  0001 C CNN
 	1    2150 2800
@@
 L Device:LED D2
 U 1 1 5B694BB9
-P 2450 4900
-F 0 "D2" V 2488 4783 50  0000 R CNN
-F 1 "LED" V 2397 4783 50  0000 R CNN
-F 2 "LED_SMD:LED_1206_3216Metric_Pad1.42x1.75mm_HandSolder" H 2450 4900 50  0001 C CNN
-F 3 "~" H 2450 4900 50  0001 C CNN
-	1    2450 4900
+P 2450 5050
+F 0 "D2" V 2488 4933 50  0000 R CNN
+F 1 "LED" V 2397 4933 50  0000 R CNN
+F 2 "LED_SMD:LED_1206_3216Metric_Pad1.42x1.75mm_HandSolder" H 2450 5050 50  0001 C CNN
+F 3 "~" H 2450 5050 50  0001 C CNN
+	1    2450 5050
 	0    -1   -1   0
 $EndComp
@@
 L Device:LED D3
 U 1 1 5B694D3F
-P 2750 4900
-F 0 "D3" V 2788 4783 50  0000 R CNN
-F 1 "LED" V 2697 4783 50  0000 R CNN
-F 2 "LED_SMD:LED_1206_3216Metric_Pad1.42x1.75mm_HandSolder" H 2750 4900 50  0001 C CNN
-F 3 "~" H 2750 4900 50  0001 C CNN
-	1    2750 4900
+P 2750 5050
+F 0 "D3" V 2788 4933 50  0000 R CNN
+F 1 "LED" V 2697 4933 50  0000 R CNN
+F 2 "LED_SMD:LED_1206_3216Metric_Pad1.42x1.75mm_HandSolder" H 2750 5050 50  0001 C CNN
+F 3 "~" H 2750 5050 50  0001 C CNN
+	1    2750 5050
 	0    -1   -1   0
 $EndComp
@@
 L Device:LED D4
 U 1 1 5B694D81
-P 3050 4900
-F 0 "D4" V 3088 4783 50  0000 R CNN
-F 1 "LED" V 2997 4783 50  0000 R CNN
-F 2 "LED_SMD:LED_1206_3216Metric_Pad1.42x1.75mm_HandSolder" H 3050 4900 50  0001 C CNN
-F 3 "~" H 3050 4900 50  0001 C CNN
-	1    3050 4900
+P 3050 5050
+F 0 "D4" V 3088 4933 50  0000 R CNN
+F 1 "LED" V 2997 4933 50  0000 R CNN
+F 2 "LED_SMD:LED_1206_3216Metric_Pad1.42x1.75mm_HandSolder" H 3050 5050 50  0001 C CNN
+F 3 "~" H 3050 5050 50  0001 C CNN
+	1    3050 5050
 	0    -1   -1   0
 $EndComp
@@
 L Device:LED D5
 U 1 1 5B694DB9
-P 3350 4900
-F 0 "D5" V 3388 4783 50  0000 R CNN
-F 1 "LED" V 3297 4783 50  0000 R CNN
-F 2 "LED_SMD:LED_1206_3216Metric_Pad1.42x1.75mm_HandSolder" H 3350 4900 50  0001 C CNN
-F 3 "~" H 3350 4900 50  0001 C CNN
-	1    3350 4900
+P 3350 5050
+F 0 "D5" V 3388 4933 50  0000 R CNN
+F 1 "LED" V 3297 4933 50  0000 R CNN
+F 2 "LED_SMD:LED_1206_3216Metric_Pad1.42x1.75mm_HandSolder" H 3350 5050 50  0001 C CNN
+F 3 "~" H 3350 5050 50  0001 C CNN
+	1    3350 5050
 	0    -1   -1   0
 $EndComp
@@
 L power:GND #PWR0109
 U 1 1 5B69FEA1
-P 2900 5250
-F 0 "#PWR0109" H 2900 5000 50  0001 C CNN
-F 1 "GND" H 2905 5077 50  0000 C CNN
-F 2 "" H 2900 5250 50  0001 C CNN
-F 3 "" H 2900 5250 50  0001 C CNN
-	1    2900 5250
-	1    0    0    -1
-$EndComp
-Wire Wire Line
-	2450 5050 2450 5250
-Wire Wire Line
-	2450 5250 2750 5250
-Wire Wire Line
-	2750 5050 2750 5250
-Connection ~ 2750 5250
-Wire Wire Line
-	2750 5250 2900 5250
-Wire Wire Line
-	2900 5250 3050 5250
-Wire Wire Line
-	3050 5250 3050 5050
-Connection ~ 2900 5250
-Wire Wire Line
-	3050 5250 3350 5250
-Wire Wire Line
-	3350 5250 3350 5050
-Connection ~ 3050 5250
-$Comp
-L Device:R R4
-U 1 1 5B6A4909
-P 2450 4600
-F 0 "R4" H 2520 4646 50  0000 L CNN
-F 1 "R" H 2520 4555 50  0000 L CNN
-F 2 "Resistor_SMD:R_1206_3216Metric_Pad1.42x1.75mm_HandSolder" V 2380 4600 50  0001 C CNN
-F 3 "~" H 2450 4600 50  0001 C CNN
-	1    2450 4600
-	1    0    0    -1
-$EndComp
-$Comp
-L Device:R R5
-U 1 1 5B6A49FF
-P 2750 4600
-F 0 "R5" H 2820 4646 50  0000 L CNN
-F 1 "R" H 2820 4555 50  0000 L CNN
-F 2 "Resistor_SMD:R_1206_3216Metric_Pad1.42x1.75mm_HandSolder" V 2680 4600 50  0001 C CNN
-F 3 "~" H 2750 4600 50  0001 C CNN
-	1    2750 4600
-	1    0    0    -1
-$EndComp
-$Comp
-L Device:R R6
-U 1 1 5B6A4A3F
-P 3050 4600
-F 0 "R6" H 3120 4646 50  0000 L CNN
-F 1 "R" H 3120 4555 50  0000 L CNN
-F 2 "Resistor_SMD:R_1206_3216Metric_Pad1.42x1.75mm_HandSolder" V 2980 4600 50  0001 C CNN
-F 3 "~" H 3050 4600 50  0001 C CNN
-	1    3050 4600
-	1    0    0    -1
-$EndComp
-$Comp
-L Device:R R7
-U 1 1 5B6A4ADD
-P 3350 4600
-F 0 "R7" H 3420 4646 50  0000 L CNN
-F 1 "R" H 3420 4555 50  0000 L CNN
-F 2 "Resistor_SMD:R_1206_3216Metric_Pad1.42x1.75mm_HandSolder" V 3280 4600 50  0001 C CNN
-F 3 "~" H 3350 4600 50  0001 C CNN
-	1    3350 4600
-	1    0    0    -1
-$EndComp
+P 2900 5400
+F 0 "#PWR0109" H 2900 5150 50  0001 C CNN
+F 1 "GND" H 2905 5227 50  0000 C CNN
+F 2 "" H 2900 5400 50  0001 C CNN
+F 3 "" H 2900 5400 50  0001 C CNN
+	1    2900 5400
+	1    0    0    -1
+$EndComp
+Wire Wire Line
+	2450 5200 2450 5400
+Wire Wire Line
+	2450 5400 2750 5400
+Wire Wire Line
+	2750 5200 2750 5400
+Connection ~ 2750 5400
+Wire Wire Line
+	2750 5400 2900 5400
+Wire Wire Line
+	2900 5400 3050 5400
+Wire Wire Line
+	3050 5400 3050 5200
+Connection ~ 2900 5400
+Wire Wire Line
+	3050 5400 3350 5400
+Wire Wire Line
+	3350 5400 3350 5200
+Connection ~ 3050 5400
 $Comp
 L Device:R R3
@@
 Text Notes 1750 4150 0    50   ~ 0
 PWR_GOOD
-Text Notes 2650 4150 0    50   ~ 0
+Text Notes 2950 4300 0    50   ~ 0
 MCU_DEBUG_LEDS
 Text Notes 1600 2000 0    50   ~ 0
@@
 L power:+3V3 #PWR0116
 U 1 1 5B6BD2D4
-P 2450 4450
-F 0 "#PWR0116" H 2450 4300 50  0001 C CNN
-F 1 "+3V3" H 2465 4623 50  0000 C CNN
-F 2 "" H 2450 4450 50  0001 C CNN
-F 3 "" H 2450 4450 50  0001 C CNN
-	1    2450 4450
-	1    0    0    -1
-$EndComp
-$Comp
-L power:+3V3 #PWR0122
-U 1 1 5B6BD35C
-P 2750 4450
-F 0 "#PWR0122" H 2750 4300 50  0001 C CNN
-F 1 "+3V3" H 2765 4623 50  0000 C CNN
-F 2 "" H 2750 4450 50  0001 C CNN
-F 3 "" H 2750 4450 50  0001 C CNN
-	1    2750 4450
-	1    0    0    -1
-$EndComp
-$Comp
-L power:+3V3 #PWR0123
-U 1 1 5B6BD3EF
-P 3050 4450
-F 0 "#PWR0123" H 3050 4300 50  0001 C CNN
-F 1 "+3V3" H 3065 4623 50  0000 C CNN
-F 2 "" H 3050 4450 50  0001 C CNN
-F 3 "" H 3050 4450 50  0001 C CNN
-	1    3050 4450
-	1    0    0    -1
-$EndComp
-$Comp
-L power:+3V3 #PWR0124
-U 1 1 5B6BD42C
-P 3350 4450
-F 0 "#PWR0124" H 3350 4300 50  0001 C CNN
-F 1 "+3V3" H 3365 4623 50  0000 C CNN
-F 2 "" H 3350 4450 50  0001 C CNN
-F 3 "" H 3350 4450 50  0001 C CNN
-	1    3350 4450
+P 2750 4350
+F 0 "#PWR0116" H 2750 4200 50  0001 C CNN
+F 1 "+3V3" H 2765 4523 50  0000 C CNN
+F 2 "" H 2750 4350 50  0001 C CNN
+F 3 "" H 2750 4350 50  0001 C CNN
+	1    2750 4350
 	1    0    0    -1
 $EndComp
@@
 NoConn ~ 8200 4600
 NoConn ~ 10250 4450
+$Comp
+L Device:R_Network04 RN1
+U 1 1 5B672BA8
+P 2950 4550
+F 0 "RN1" H 3130 4596 50  0000 L CNN
+F 1 "R_Network04" H 3130 4505 50  0000 L CNN
+F 2 "Resistor_SMD:R_Array_Convex_4x1206" V 3225 4550 50  0001 C CNN
+F 3 "http://www.vishay.com/docs/31509/csc.pdf" H 2950 4550 50  0001 C CNN
+	1    2950 4550
+	1    0    0    -1
+$EndComp
+Wire Wire Line
+	2750 4750 2450 4750
+Wire Wire Line
+	2450 4750 2450 4900
+Wire Wire Line
+	2850 4750 2850 4850
+Wire Wire Line
+	2850 4850 2750 4850
+Wire Wire Line
+	2750 4850 2750 4900
+Wire Wire Line
+	2950 4750 2950 4850
+Wire Wire Line
+	2950 4850 3050 4850
+Wire Wire Line
+	3050 4850 3050 4900
+Wire Wire Line
+	3050 4750 3350 4750
+Wire Wire Line
+	3350 4750 3350 4900
 $EndSCHEMATC

Commit message: sch: LED_DBUGn
Signed-off-by: Ben Lancaster <bdl@live.co.uk>
Parts:
- removed RN1: R_Network04, Resistor_SMD:R_Array_Convex_4x1206, symbol Device:R_Network04
- added R4, R5, R6, R7: 50, Resistor_SMD:R_0603_1608Metric_Pad1.05x0.95mm_HandSolder, symbol Device:R
Connections:
- net labels added: LED_DBUG1, LED_DBUG2, LED_DBUG3, LED_DBUG4
- wire segments 73 -> 67
- no-connect marks 16 -> 12
Changed lines of the file:
@@
 Text GLabel 3900 2200 2    50   Input ~ 0
 ADC_IN0
-Text GLabel 3900 2300 2    50   Input ~ 0
-ADC_IN1
 $Comp
 L Connector_Generic:Conn_02x08_Odd_Even J4
@@
 	8100 5300 8400 5300
 NoConn ~ 2600 3300
-NoConn ~ 3900 2400
-NoConn ~ 3900 2500
-NoConn ~ 3900 2600
 NoConn ~ 3900 2700
 NoConn ~ 3900 2800
@@
 L Device:LED D2
 U 1 1 5B694BB9
-P 2450 5050
-F 0 "D2" V 2488 4933 50  0000 R CNN
-F 1 "LED" V 2397 4933 50  0000 R CNN
-F 2 "LED_SMD:LED_1206_3216Metric_Pad1.42x1.75mm_HandSolder" H 2450 5050 50  0001 C CNN
-F 3 "~" H 2450 5050 50  0001 C CNN
-	1    2450 5050
+P 3250 5400
+F 0 "D2" V 3288 5283 50  0000 R CNN
+F 1 "LED" V 3197 5283 50  0000 R CNN
+F 2 "LED_SMD:LED_1206_3216Metric_Pad1.42x1.75mm_HandSolder" H 3250 5400 50  0001 C CNN
+F 3 "~" H 3250 5400 50  0001 C CNN
+	1    3250 5400
 	0    -1   -1   0
 $EndComp
@@
 L Device:LED D3
 U 1 1 5B694D3F
-P 2750 5050
-F 0 "D3" V 2788 4933 50  0000 R CNN
-F 1 "LED" V 2697 4933 50  0000 R CNN
-F 2 "LED_SMD:LED_1206_3216Metric_Pad1.42x1.75mm_HandSolder" H 2750 5050 50  0001 C CNN
-F 3 "~" H 2750 5050 50  0001 C CNN
-	1    2750 5050
+P 3550 5400
+F 0 "D3" V 3588 5283 50  0000 R CNN
+F 1 "LED" V 3497 5283 50  0000 R CNN
+F 2 "LED_SMD:LED_1206_3216Metric_Pad1.42x1.75mm_HandSolder" H 3550 5400 50  0001 C CNN
+F 3 "~" H 3550 5400 50  0001 C CNN
+	1    3550 5400
 	0    -1   -1   0
 $EndComp
@@
 L Device:LED D4
 U 1 1 5B694D81
-P 3050 5050
-F 0 "D4" V 3088 4933 50  0000 R CNN
-F 1 "LED" V 2997 4933 50  0000 R CNN
-F 2 "LED_SMD:LED_1206_3216Metric_Pad1.42x1.75mm_HandSolder" H 3050 5050 50  0001 C CNN
-F 3 "~" H 3050 5050 50  0001 C CNN
-	1    3050 5050
+P 3850 5400
+F 0 "D4" V 3888 5283 50  0000 R CNN
+F 1 "LED" V 3797 5283 50  0000 R CNN
+F 2 "LED_SMD:LED_1206_3216Metric_Pad1.42x1.75mm_HandSolder" H 3850 5400 50  0001 C CNN
+F 3 "~" H 3850 5400 50  0001 C CNN
+	1    3850 5400
 	0    -1   -1   0
 $EndComp
@@
 L Device:LED D5
 U 1 1 5B694DB9
-P 3350 5050
-F 0 "D5" V 3388 4933 50  0000 R CNN
-F 1 "LED" V 3297 4933 50  0000 R CNN
-F 2 "LED_SMD:LED_1206_3216Metric_Pad1.42x1.75mm_HandSolder" H 3350 5050 50  0001 C CNN
-F 3 "~" H 3350 5050 50  0001 C CNN
-	1    3350 5050
+P 4150 5400
+F 0 "D5" V 4188 5283 50  0000 R CNN
+F 1 "LED" V 4097 5283 50  0000 R CNN
+F 2 "LED_SMD:LED_1206_3216Metric_Pad1.42x1.75mm_HandSolder" H 4150 5400 50  0001 C CNN
+F 3 "~" H 4150 5400 50  0001 C CNN
+	1    4150 5400
 	0    -1   -1   0
 $EndComp
@@
 L power:GND #PWR0109
 U 1 1 5B69FEA1
-P 2900 5400
-F 0 "#PWR0109" H 2900 5150 50  0001 C CNN
-F 1 "GND" H 2905 5227 50  0000 C CNN
-F 2 "" H 2900 5400 50  0001 C CNN
-F 3 "" H 2900 5400 50  0001 C CNN
-	1    2900 5400
-	1    0    0    -1
-$EndComp
-Wire Wire Line
-	2450 5200 2450 5400
-Wire Wire Line
-	2450 5400 2750 5400
-Wire Wire Line
-	2750 5200 2750 5400
-Connection ~ 2750 5400
-Wire Wire Line
-	2750 5400 2900 5400
-Wire Wire Line
-	2900 5400 3050 5400
-Wire Wire Line
-	3050 5400 3050 5200
-Connection ~ 2900 5400
-Wire Wire Line
-	3050 5400 3350 5400
-Wire Wire Line
-	3350 5400 3350 5200
-Connection ~ 3050 5400
+P 3700 5750
+F 0 "#PWR0109" H 3700 5500 50  0001 C CNN
+F 1 "GND" H 3705 5577 50  0000 C CNN
+F 2 "" H 3700 5750 50  0001 C CNN
+F 3 "" H 3700 5750 50  0001 C CNN
+	1    3700 5750
+	1    0    0    -1
+$EndComp
+Wire Wire Line
+	3250 5550 3250 5750
+Wire Wire Line
+	3250 5750 3550 5750
+Wire Wire Line
+	3550 5550 3550 5750
+Connection ~ 3550 5750
+Wire Wire Line
+	3550 5750 3700 5750
+Wire Wire Line
+	3700 5750 3850 5750
+Wire Wire Line
+	3850 5750 3850 5550
+Connection ~ 3700 5750
+Wire Wire Line
+	3850 5750 4150 5750
+Wire Wire Line
+	4150 5750 4150 5550
+Connection ~ 3850 5750
 $Comp
 L Device:R R3
@@
 Text Notes 1750 4150 0    50   ~ 0
 PWR_GOOD
-Text Notes 2950 4300 0    50   ~ 0
+Text Notes 3400 4250 0    50   ~ 0
 MCU_DEBUG_LEDS
 Text Notes 1600 2000 0    50   ~ 0
@@
 Text GLabel 10350 4450 2    50   Input ~ 0
 FPGA_3V3
-$Comp
-L power:+3V3 #PWR0116
-U 1 1 5B6BD2D4
-P 2750 4350
-F 0 "#PWR0116" H 2750 4200 50  0001 C CNN
-F 1 "+3V3" H 2765 4523 50  0000 C CNN
-F 2 "" H 2750 4350 50  0001 C CNN
-F 3 "" H 2750 4350 50  0001 C CNN
-	1    2750 4350
-	1    0    0    -1
-$EndComp
 NoConn ~ 3900 2200
-NoConn ~ 3900 2300
 NoConn ~ 8400 5200
 NoConn ~ 8400 5300
@@
 NoConn ~ 8200 4600
 NoConn ~ 10250 4450
-$Comp
-L Device:R_Network04 RN1
-U 1 1 5B672BA8
-P 2950 4550
-F 0 "RN1" H 3130 4596 50  0000 L CNN
-F 1 "R_Network04" H 3130 4505 50  0000 L CNN
-F 2 "Resistor_SMD:R_Array_Convex_4x1206" V 3225 4550 50  0001 C CNN
-F 3 "http://www.vishay.com/docs/31509/csc.pdf" H 2950 4550 50  0001 C CNN
-	1    2950 4550
-	1    0    0    -1
-$EndComp
-Wire Wire Line
-	2750 4750 2450 4750
-Wire Wire Line
-	2450 4750 2450 4900
-Wire Wire Line
-	2850 4750 2850 4850
-Wire Wire Line
-	2850 4850 2750 4850
-Wire Wire Line
-	2750 4850 2750 4900
-Wire Wire Line
-	2950 4750 2950 4850
-Wire Wire Line
-	2950 4850 3050 4850
-Wire Wire Line
-	3050 4850 3050 4900
-Wire Wire Line
-	3050 4750 3350 4750
-Wire Wire Line
-	3350 4750 3350 4900
+Wire Wire Line
+	3250 5100 3250 5250
+Wire Wire Line
+	4150 5100 4150 5250
+$Comp
+L Device:R R4
+U 1 1 5B676B30
+P 3250 4950
+F 0 "R4" H 3320 4996 50  0000 L CNN
+F 1 "50" H 3320 4905 50  0000 L CNN
+F 2 "Resistor_SMD:R_0603_1608Metric_Pad1.05x0.95mm_HandSolder" V 3180 4950 50  0001 C CNN
+F 3 "~" H 3250 4950 50  0001 C CNN
+	1    3250 4950
+	1    0    0    -1
+$EndComp
+Wire Wire Line
+	3850 5100 3850 5250
+Wire Wire Line
+	3550 5100 3550 5250
+Text GLabel 3900 2600 2    50   Input ~ 0
+LED_DBUG1
+Text GLabel 3900 2500 2    50   Input ~ 0
+LED_DBUG2
+Text GLabel 3900 2400 2    50   Input ~ 0
+LED_DBUG3
+Text GLabel 3900 2300 2    50   Input ~ 0
+LED_DBUG4
+Text GLabel 3250 4800 1    50   Input ~ 0
+LED_DBUG1
+Text GLabel 3550 4800 1    50   Input ~ 0
+LED_DBUG2
+Text GLabel 3850 4800 1    50   Input ~ 0
+LED_DBUG3
+Text GLabel 4150 4800 1    50   Input ~ 0
+LED_DBUG4
+$Comp
+L Device:R R5
+U 1 1 5B67EFB9
+P 3550 4950
+F 0 "R5" H 3620 4996 50  0000 L CNN
+F 1 "50" H 3620 4905 50  0000 L CNN
+F 2 "Resistor_SMD:R_0603_1608Metric_Pad1.05x0.95mm_HandSolder" V 3480 4950 50  0001 C CNN
+F 3 "~" H 3550 4950 50  0001 C CNN
+	1    3550 4950
+	1    0    0    -1
+$EndComp
+$Comp
+L Device:R R6
+U 1 1 5B67EFFF
+P 3850 4950
+F 0 "R6" H 3920 4996 50  0000 L CNN
+F 1 "50" H 3920 4905 50  0000 L CNN
+F 2 "Resistor_SMD:R_0603_1608Metric_Pad1.05x0.95mm_HandSolder" V 3780 4950 50  0001 C CNN
+F 3 "~" H 3850 4950 50  0001 C CNN
+	1    3850 4950
+	1    0    0    -1
+$EndComp
+$Comp
+L Device:R R7
+U 1 1 5B67F047
+P 4150 4950
+F 0 "R7" H 4220 4996 50  0000 L CNN
+F 1 "50" H 4220 4905 50  0000 L CNN
+F 2 "Resistor_SMD:R_0603_1608Metric_Pad1.05x0.95mm_HandSolder" V 4080 4950 50  0001 C CNN
+F 3 "~" H 4150 4950 50  0001 C CNN
+	1    4150 4950
+	1    0    0    -1
+$EndComp
 $EndSCHEMATC

Commit message: pcb: Connected LEDs and I2Cs
Signed-off-by: Ben Lancaster <bdl@live.co.uk>
Changed lines of the file:
@@
 Text GLabel 3900 2300 2    50   Input ~ 0
 LED_DBUG4
+Text GLabel 4150 4800 1    50   Input ~ 0
+LED_DBUG1
+Text GLabel 3850 4800 1    50   Input ~ 0
+LED_DBUG2
+Text GLabel 3550 4800 1    50   Input ~ 0
+LED_DBUG3
 Text GLabel 3250 4800 1    50   Input ~ 0
-LED_DBUG1
-Text GLabel 3550 4800 1    50   Input ~ 0
-LED_DBUG2
-Text GLabel 3850 4800 1    50   Input ~ 0
-LED_DBUG3
-Text GLabel 4150 4800 1    50   Input ~ 0
 LED_DBUG4
 $Comp

Commit message: pcb: Flip stlink connector to prevent clash with 5 pin header
Signed-off-by: Ben <bdl@live.co.uk>
Parts:
- R4, R5, R6, R7: value 50 -> 100
Connections:
- wire segments 67 -> 68
Other:
- moved on the sheet: U2
Changed lines of the file:
@@
 L Regulator_Linear:LD1117S33TR_SOT223 U2
 U 1 1 5B61E64C
-P 5350 950
-F 0 "U2" H 5350 1192 50  0000 C CNN
-F 1 "LD1117S33TR_SOT223" H 5350 1101 50  0000 C CNN
-F 2 "Package_TO_SOT_SMD:SOT-223-3_TabPin2" H 5350 1150 50  0001 C CNN
-F 3 "http://www.st.com/st-web-ui/static/active/en/resource/technical/document/datasheet/CD00000544.pdf" H 5450 700 50  0001 C CNN
-	1    5350 950
+P 5400 1100
+F 0 "U2" H 5400 1342 50  0000 C CNN
+F 1 "LD1117S33TR_SOT223" H 5400 1251 50  0000 C CNN
+F 2 "Package_TO_SOT_SMD:SOT-223-3_TabPin2" H 5400 1300 50  0001 C CNN
+F 3 "http://www.st.com/st-web-ui/static/active/en/resource/technical/document/datasheet/CD00000544.pdf" H 5500 850 50  0001 C CNN
+	1    5400 1100
 	-1   0    0    -1
 $EndComp
@@
 L power:+5V #PWR0108
 U 1 1 5B61EA0F
-P 5950 950
-F 0 "#PWR0108" H 5950 800 50  0001 C CNN
-F 1 "+5V" H 5965 1123 50  0000 C CNN
-F 2 "" H 5950 950 50  0001 C CNN
-F 3 "" H 5950 950 50  0001 C CNN
-	1    5950 950
-	1    0    0    -1
-$EndComp
-Wire Wire Line
-	5650 950  5950 950
-Wire Wire Line
-	4750 950  5050 950
+P 6000 1100
+F 0 "#PWR0108" H 6000 950 50  0001 C CNN
+F 1 "+5V" H 6015 1273 50  0000 C CNN
+F 2 "" H 6000 1100 50  0001 C CNN
+F 3 "" H 6000 1100 50  0001 C CNN
+	1    6000 1100
+	1    0    0    -1
+$EndComp
+Wire Wire Line
+	5700 1100 6000 1100
+Wire Wire Line
+	4800 1100 5100 1100
 $Comp
 L power:GND #PWR0110
 U 1 1 5B61ED16
-P 5350 1250
-F 0 "#PWR0110" H 5350 1000 50  0001 C CNN
-F 1 "GND" H 5355 1077 50  0000 C CNN
-F 2 "" H 5350 1250 50  0001 C CNN
-F 3 "" H 5350 1250 50  0001 C CNN
-	1    5350 1250
+P 5400 1400
+F 0 "#PWR0110" H 5400 1150 50  0001 C CNN
+F 1 "GND" H 5405 1227 50  0000 C CNN
+F 2 "" H 5400 1400 50  0001 C CNN
+F 3 "" H 5400 1400 50  0001 C CNN
+	1    5400 1400
 	1    0    0    -1
 $EndComp
@@
 L power:GND #PWR0109
 U 1 1 5B69FEA1
-P 3700 5750
-F 0 "#PWR0109" H 3700 5500 50  0001 C CNN
-F 1 "GND" H 3705 5577 50  0000 C CNN
-F 2 "" H 3700 5750 50  0001 C CNN
-F 3 "" H 3700 5750 50  0001 C CNN
-	1    3700 5750
+P 3700 5850
+F 0 "#PWR0109" H 3700 5600 50  0001 C CNN
+F 1 "GND" H 3705 5677 50  0000 C CNN
+F 2 "" H 3700 5850 50  0001 C CNN
+F 3 "" H 3700 5850 50  0001 C CNN
+	1    3700 5850
 	1    0    0    -1
 $EndComp
@@
 Text GLabel 6750 1050 0    50   Input ~ 0
 STLINK_3V3
-Text GLabel 4750 950  1    50   Input ~ 0
+Text GLabel 4800 1100 1    50   Input ~ 0
 BOARD_3V3
 Text GLabel 6750 1250 0    50   Input ~ 0
@@
 P 3250 4950
 F 0 "R4" H 3320 4996 50  0000 L CNN
-F 1 "50" H 3320 4905 50  0000 L CNN
+F 1 "100" H 3320 4905 50  0000 L CNN
 F 2 "Resistor_SMD:R_0603_1608Metric_Pad1.05x0.95mm_HandSolder" V 3180 4950 50  0001 C CNN
 F 3 "~" H 3250 4950 50  0001 C CNN
@@
 P 3550 4950
 F 0 "R5" H 3620 4996 50  0000 L CNN
-F 1 "50" H 3620 4905 50  0000 L CNN
+F 1 "100" H 3620 4905 50  0000 L CNN
 F 2 "Resistor_SMD:R_0603_1608Metric_Pad1.05x0.95mm_HandSolder" V 3480 4950 50  0001 C CNN
 F 3 "~" H 3550 4950 50  0001 C CNN
@@
 P 3850 4950
 F 0 "R6" H 3920 4996 50  0000 L CNN
-F 1 "50" H 3920 4905 50  0000 L CNN
+F 1 "100" H 3920 4905 50  0000 L CNN
 F 2 "Resistor_SMD:R_0603_1608Metric_Pad1.05x0.95mm_HandSolder" V 3780 4950 50  0001 C CNN
 F 3 "~" H 3850 4950 50  0001 C CNN
@@
 P 4150 4950
 F 0 "R7" H 4220 4996 50  0000 L CNN
-F 1 "50" H 4220 4905 50  0000 L CNN
+F 1 "100" H 4220 4905 50  0000 L CNN
 F 2 "Resistor_SMD:R_0603_1608Metric_Pad1.05x0.95mm_HandSolder" V 4080 4950 50  0001 C CNN
 F 3 "~" H 4150 4950 50  0001 C CNN
@@
 	1    0    0    -1
 $EndComp
+Wire Wire Line
+	3700 5750 3700 5850
 $EndSCHEMATC

Commit message: pcb: Resize to exactly 1x2 inches to save on costs
Signed-off-by: Ben Lancaster <bdl@live.co.uk>
Parts:
- R3: value R -> 100
Changed lines of the file:
@@
 P 1950 4550
 F 0 "R3" H 2020 4596 50  0000 L CNN
-F 1 "R" H 2020 4505 50  0000 L CNN
+F 1 "100" H 2020 4505 50  0000 L CNN
 F 2 "Resistor_SMD:R_1206_3216Metric_Pad1.42x1.75mm_HandSolder" V 1880 4550 50  0001 C CNN
 F 3 "~" H 1950 4550 50  0001 C CNN
